Commit message: Preparing LiDAR implementation for testing

File: launch/includes/hokuyo.urdf.xacro (robot description, xacro)
@@ -13,5 +13,5 @@
         <origin xyz="0 0 0" rpy="0 0 0"/>
         <geometry>
-          <mesh filename="package://turtlebot_description/meshes/sensors/hokuyo.dae"/>
+          <mesh filename="$(find fgm_plugin)/launch/includes/hokuyo.dae"/>
         </geometry>
       </visual>

Commit message: Revert "Lidar fov"

File: launch/includes/hokuyo.urdf.xacro (robot description, xacro)
@@ -13,5 +13,5 @@
         <origin xyz="0 0 0" rpy="0 0 0"/>
         <geometry>
-          <mesh filename="$(find fgm_plugin)/launch/includes/hokuyo.dae"/>
+          <mesh filename="package://turtlebot_description/meshes/sensors/hokuyo.dae"/>
         </geometry>
       </visual>
